File: hardware/distance-us-v2-bricklet.kicad_pcb (KiCad board)
At the start: 2 copper layers, 30 x 30 mm, 22 parts, among them P1 CON-SENSOR2, P2 DEBUG, P3 BOOT, U1 XMC1XXX24, U2 DRILL, U3 DRILL, U4 DRILL, U5 DRILL, U6 HRLV-EZ

Commit message: changed schematic
Parts:
- added G***: Logo_31x31, kicad-libraries:Logo_31x31, B.Cu at (151.6, 95.5)
- added G***: LOGO, kicad-libraries:Logo_CoMCU, B.Cu at (150.0, 104.6)
- added VAL: WEEE_7mm, kicad-libraries:WEEE_7mm, B.Cu at (141.5, 105.4)
- added VAL: CE_5mm, kicad-libraries:CE_5mm, B.Cu at (158.5, 104.6)
- moved L1 1.64 mm to (147.7, 102.8), turned to 90 degrees
- moved RP2 0.30 mm to (150.0, 90.0)
Routing:
- net 3V3: track 68.2 -> 72.6 mm, vias 4 -> 6
- net GND: track 31.6 -> 35.0 mm
- net Net-(P2-Pad1): track 11.5 -> 12.0 mm
Other:
- board text added: "Distance"
- board text added: "Distance US 2.0"
- board text added: "Status"
- board text added: "tinkerforge.com"
